Commit message: feat[add+update] : ellie arm + urdf "echo 1 | sudo tee /sys/bus/usbserial/devices/ttyUSB0/latency_timer add : Ros2 interfaces

File: src/ellie_arm/urdf/ellie.urdf (robot description, URDF)
Before this commit: robot Poppy_Torso, 14 links, 13 joints
Links:
- link base: geometry collision mesh filename=package://urdf/meshes/base_respondable.STL; visual mesh filename=package://urdf/meshes/base_visual.STL
- link bust_motors: geometry collision mesh filename=package://urdf/meshes/bust_motors_respondable.STL; visual mesh filename=package://urdf/meshes/bust_motors_visual.STL
- link chest: geometry collision mesh filename=package://urdf/meshes/chest_respondable.STL; visual mesh filename=package://urdf/meshes/chest_visual.STL
- link head: geometry collision mesh filename=package://urdf/meshes/head_respondable.STL; visual mesh filename=package://urdf/meshes/head_visual.STL
- link l_forearm: geometry collision mesh filename=package://urdf/meshes/l_forearm_respondable.STL; visual mesh filename=package://urdf/meshes/l_forearm_visual.STL
- link l_shoulder: geometry collision mesh filename=package://urdf/meshes/l_shoulder_respondable.STL; visual mesh filename=package://urdf/meshes/l_shoulder_visual.STL
- link l_shoulder_motor: geometry collision mesh filename=package://urdf/meshes/l_shoulder_motor_respondable.STL; visual mesh filename=package://urdf/meshes/l_shoulder_motor_visual.STL
- link l_upper_arm: geometry collision mesh filename=package://urdf/meshes/l_upper_arm_respondable.STL; visual mesh filename=package://urdf/meshes/l_upper_arm_visual.STL
- link neck: geometry collision mesh filename=package://urdf/meshes/neck_respondable.STL; visual mesh filename=package://urdf/meshes/neck_visual.STL
- link r_forearm: geometry collision mesh filename=package://urdf/meshes/r_forearm_respondable.STL; visual mesh filename=package://urdf/meshes/r_forearm_visual.STL
- link r_shoulder: geometry collision mesh filename=package://urdf/meshes/r_shoulder_respondable.STL; visual mesh filename=package://urdf/meshes/r_shoulder_visual.STL
- link r_shoulder_motor: geometry collision mesh filename=package://urdf/meshes/r_shoulder_motor_respondable.STL; visual mesh filename=package://urdf/meshes/r_shoulder_motor_visual.STL
- link r_upper_arm: geometry collision mesh filename=package://urdf/meshes/r_upper_arm_respondable.STL; visual mesh filename=package://urdf/meshes/r_upper_arm_visual.STL
- link spine: geometry collision mesh filename=package://urdf/meshes/spine_respondable.STL; visual mesh filename=package://urdf/meshes/spine_visual.STL
